File: kicad/scart2dvi.kicad_pcb (KiCad board)
At the start: 2 copper layers, 108 x 82 mm, 54 parts, among them J1 Micro USB, J2 SCART-F, J3 SJ-3523-SMT-TR, J4 0743201004, Q1 MMBT3906, Q2 MMBT3906, SW1 SW_SPDT, SW2 SW_SPDT, U1 THS7368, U2 LMH1980

Commit message: pull down disable pins
Connections:
- net Net-(R10-Pad2) renamed /VIDEO_AMP/480p
- net Net-(R9-Pad2) renamed /VIDEO_AMP/FILTER_OFF
- U1 pad 15: Net-(U1-Pad15) -> GND
- U1 pad 17: Net-(U1-Pad17) -> GND
